Commit message: first commit

File: src/rover_description/urdf/robot.xacro (robot description, xacro)
@@ -9,9 +9,9 @@
   <xacro:property name="wheel_r" value="0.05"/>  <!-- radius -->
   <xacro:property name="wheel_w" value="0.08"/>  <!-- width -->
-  <xacro:property name="clearance" value="0.25"/>  <!-- 250 mm -->
+  <xacro:property name="clearance" value="0.215"/>  <!-- 215 mm -->
   <!-- Slight outside offset so wheels stick out correctly -->
-  <xacro:property name="wheel_y_offset" value="${W/2 + 0.02}"/>
-  <xacro:property name="wheel_x_front" value="${L/2 - 0.06}"/>
-  <xacro:property name="wheel_x_back"  value="-${L/2 - 0.06}"/>
+  <xacro:property name="wheel_y_offset" value="${W/2 + wheel_w/2 + 0.02}"/>
+  <xacro:property name="wheel_x_front" value="${L/2 + 0.04}"/>
+  <xacro:property name="wheel_x_back"  value="-${L/2 + 0.02}"/>
   <!-- ========================= -->
   <!-- Physical Material + Mass  -->
@@ -66,49 +66,49 @@
   <!-- WHEEL MACRO -->
   <!-- ========================= -->
-  <xacro:macro name="wheel" params="wheel_name x y">
-  <link name="${wheel_name}_link">
-    <visual>
-      <!-- rotate cylinder so its axis aligns with the joint axis (y) -->
-      <origin xyz="0 0 0" rpy="-1.57 0 0"/>
-      <geometry>
-        <cylinder radius="${wheel_r}" length="${wheel_w}"/>
-      </geometry>
-      <material name="black"><color rgba="0.1 0.1 0.1 1"/></material>
-    </visual>
-    <collision>
-      <!-- same rotation for collision geometry -->
-      <origin xyz="0 0 0" rpy="-1.57 0 0"/>
-      <geometry>
-        <cylinder radius="${wheel_r}" length="${wheel_w}"/>
-      </geometry>
-    </collision>
-    <inertial>
-      <!-- inertial principal axes rotated to match geometry orientation -->
-      <origin xyz="0 0 0" rpy="-1.57 0 0"/>
-      <mass value="${m_wheel}"/>
-      <inertia ixx="${I_wheel_axial}" ixy="0" ixz="0"
-               iyy="${I_wheel_axial}" iyz="0"
-               izz="${I_wheel_zz}"/>
-    </inertial>
-  </link>
-  <joint name="${wheel_name}_joint" type="continuous">
-    <origin xyz="${x} ${y} ${wheel_r}" rpy="0 0 0"/>
-    <parent link="base_link"/>
-    <child link="${wheel_name}_link"/>
-    <axis xyz="0 1 0"/>
-    <dynamics damping="0.1" friction="0.1"/>
-  </joint>
+  <xacro:macro name="wheel" params="wheel_name x y mesh_stl mesh_rpy joint_axis">
+    <link name="${wheel_name}_link">
+      <visual>
+        <!-- apply mesh_rpy only here (no extra implicit rotations) -->
+        <origin xyz="0 0 0" rpy="${mesh_rpy}"/>
+        <geometry>
+          <mesh filename="${mesh_stl}"/>
+        </geometry>
+      </visual>
+      <collision>
+        <!-- approximate collision as cylinder so collisions behave nicely -->
+        <!-- collision origin rotated to put cylinder axis aligned with joint axis if needed -->
+        <origin xyz="0 0 0" rpy="${mesh_rpy}"/>
+        <geometry>
+          <cylinder radius="${wheel_r}" length="${wheel_w}"/>
+        </geometry>
+      </collision>
+      <inertial>
+        <origin xyz="0 0 0" rpy="${mesh_rpy}"/>
+        <mass value="${m_wheel}"/>
+        <!-- simple wheel inertia -->
+        <inertia ixx="0.00089" ixy="0" ixz="0" iyy="0.00089" iyz="0" izz="0.0013057"/>
+      </inertial>
+    </link>
+    <joint name="${wheel_name}_joint" type="continuous">
+      <!-- joint placed at the wheel contact point: z set to wheel_r -->
+      <!-- joint origin uses x,y from macro + wheel_r -->
+      <origin xyz="${x} ${y} ${wheel_r}" rpy="0 0 0"/>
+      <parent link="base_link"/>
+      <child link="${wheel_name}_link"/>
+      <!-- allow the user-supplied axis for the joint -->
+      <axis xyz="${joint_axis}"/>
+      <dynamics damping="0.1" friction="0.1"/>
+    </joint>
   </xacro:macro>
   <!-- LiDAR link (visual/collision/inertial only) -->
   <link name="lidar_link">
     <visual>
-      <origin xyz="0 0 0" rpy="0 1.5708 0"/>
-      <geometry>
-        <cylinder radius="0.065" length="0.05"/>
-      </geometry>
-      <material name="black"><color rgba="0.1 0.1 0.1 1"/></material>
+      <origin xyz="0 0 0" rpy="3.14159 0 0"/>
+      <geometry>
+          <mesh filename="package://rover_description/meshes/Lidar.STL" scale="1 1 1"/>
+      </geometry>
     </visual>
     <collision>
-      <origin xyz="0 0 0" rpy="0 1.5708 0"/>
+      <origin xyz="0 0 0" rpy="3.14159 0 0"/>
       <geometry>
         <cylinder radius="0.065" length="0.05"/>
@@ -117,5 +117,5 @@
     <inertial>
       <mass value="0.3"/>
-      <origin xyz="0 0 0" rpy="0 1.5708 0"/>
+      <origin xyz="0 0 0" rpy="3.14159 0 0"/>
       <inertia ixx="0.001" ixy="0.0" ixz="0.0" iyy="0.001" iyz="0.0" izz="0.001"/>
     </inertial>
@@ -126,5 +126,5 @@
     <child link="lidar_link"/>
     <!-- Mount at front-center of rover, facing forward horizontally -->
-    <origin xyz="0.20 0 0.32" rpy="0 0 0"/>
+    <origin xyz="0.13 0.01 0.24" rpy="0 0 0"/>
   </joint>
   <!-- Camera link + optical frame -->
@@ -170,19 +170,31 @@
   <!-- ========================= -->
   <!-- Front Left -->
-  <xacro:wheel wheel_name="front_left"
-               x="${wheel_x_front}"
-               y="${wheel_y_offset}"/>
+    <xacro:wheel wheel_name="front_left"
+                    x="${wheel_x_front}"
+                    y="${wheel_y_offset}"
+                    mesh_stl="package://rover_description/meshes/wheel4.STL"
+                    mesh_rpy="-1.57 0 0"
+                    joint_axis="0 0 1"/>
   <!-- Front Right -->
-  <xacro:wheel wheel_name="front_right"
-               x="${wheel_x_front}"
-               y="-${wheel_y_offset}"/>
-  <!-- Rear Left -->
-  <xacro:wheel wheel_name="rear_left"
-               x="${wheel_x_back}"
-               y="${wheel_y_offset}"/>
-  <!-- Rear Right -->
-  <xacro:wheel wheel_name="rear_right"
-               x="${wheel_x_back}"
-               y="-${wheel_y_offset}"/>
+    <xacro:wheel wheel_name="front_right"
+                    x="${wheel_x_front}"
+                    y="-${wheel_y_offset}"
+                    mesh_stl="package://rover_description/meshes/wheel2.STL"
+                    mesh_rpy="-1.57 0 0"
+                    joint_axis="0 0 1"/>
+    <!-- Rear Left -->
+    <xacro:wheel wheel_name="rear_left"
+                    x="${wheel_x_back}"
+                    y="${wheel_y_offset}"
+                    mesh_stl="package://rover_description/meshes/wheel3.STL"
+                    mesh_rpy="-1.57 0 0"
+                    joint_axis="0 0 1"/>
+    <!-- Rear Right -->
+    <xacro:wheel wheel_name="rear_right"
+                    x="${wheel_x_back}"
+                    y="-${wheel_y_offset}"
+                    mesh_stl="package://rover_description/meshes/wheel1.STL"
+                    mesh_rpy="-1.57 0 0"
+                    joint_axis="0 0 1"/>
   <!-- ========================= -->
   <!-- GAZEBO PLUGINS (Inline for Harmonic) -->

Commit message: Remove teleop launch, update RViz condition, and adjust front wheel x-offset in URDF.

File: src/rover_description/urdf/robot.xacro (robot description, xacro)
@@ -12,5 +12,5 @@
   <!-- Slight outside offset so wheels stick out correctly -->
   <xacro:property name="wheel_y_offset" value="${W/2 + wheel_w/2 + 0.02}"/>
-  <xacro:property name="wheel_x_front" value="${L/2 + 0.04}"/>
+  <xacro:property name="wheel_x_front" value="${L/2 + 0.03}"/>
   <xacro:property name="wheel_x_back"  value="-${L/2 + 0.02}"/>
   <!-- ========================= -->

Commit message: Localization setup without the imu device || incomplete

File: src/rover_description/urdf/robot.xacro (robot description, xacro)
@@ -62,4 +62,32 @@
     <parent link="base_footprint"/>
     <child link="base_link"/>
+  </joint>
+  <!-- ========================= -->
+  <!-- IMU LINK -->
+  <!-- ========================= -->
+  <link name="imu_link">
+    <visual>
+      <origin xyz="0 0 0" rpy="0 0 0"/>
+      <geometry>
+        <box size="0.08 0.05 0.04"/>
+      </geometry>
+      <material name="black"><color rgba="0.0 0.0 0.0 1"/></material>
+    </visual>
+    <collision>
+      <origin xyz="0 0 0" rpy="0 0 0"/>
+      <geometry>
+        <box size="0.08 0.05 0.04"/>
+      </geometry>
+    </collision>
+    <inertial>
+      <mass value="0.2"/>
+      <origin xyz="0 0 0" rpy="0 0 0"/>
+      <inertia ixx="0.0005" ixy="0.0" ixz="0.0" iyy="0.0005" iyz="0.0" izz="0.0005"/>
+    </inertial>
+  </link>
+  <joint name="imu_joint" type="fixed">
+    <parent link="base_link"/>
+    <child link="imu_link"/>
+    <origin xyz="0.13 0.01 0.24" rpy="0 0 0"/>
   </joint>
   <!-- ========================= -->

Commit message: Fixing twistmux, topics, and tf flow errorts...

File: src/rover_description/urdf/robot.xacro (robot description, xacro)
@@ -1,2 +1,28 @@
+<!--I need to make sure a few things :
+the lidar_link visuals is flipped | pi value present, need to change that
+| The lidar z height is at 0.24, which is not good, need to change it :
+In your current code:
+- clearance is 0.1325 (Ground to bottom of chassis).
+- wheel_r is 0.05.
+- lidar_joint origin is at z="0.24".
+This means your LiDAR is positioned 0.24 meters above the base_link origin.
+The Problem: In your base_link visual/collision tags, you have the box offset by ${wheel_r + clearance + H/2}. In ROS, the base_link origin should ideally be on the floor or the center of the axles. Your current setup has the LiDAR floating quite high.
+The Fix: Use a relative property for the Lidar height so that when the chassis moves, the Lidar moves with it.
+and the imu:
+You have the IMU at xyz="0.13 0.01 0.24".
+As we discussed, if the IMU is offset from the center, the EKF has to do complex math to compensate for the "swing" when the robot rotates.
+The Fix: Move it to 0 0 0 (relative to the chassis) for now.
+updated code u can use:
+<joint name="imu_joint" type="fixed">
+    <parent link="base_link"/>
+    <child link="imu_link"/>
+    <origin xyz="0 0 0.05" rpy="0 0 0"/>
+  </joint>
+  <joint name="lidar_joint" type="fixed">
+    <parent link="base_link"/>
+    <child link="lidar_link"/>
+    <origin xyz="0.13 0 0.20" rpy="0 0 0"/>
+  </joint>
+-->
 <?xml version="1.0"?>
 <robot xmlns:xacro="http://www.ros.org/wiki/xacro" name="four_wheel_rover">
@@ -9,5 +35,5 @@
   <xacro:property name="wheel_r" value="0.05"/>  <!-- radius -->
   <xacro:property name="wheel_w" value="0.08"/>  <!-- width -->
-  <xacro:property name="clearance" value="0.215"/>  <!-- 215 mm -->
+  <xacro:property name="clearance" value="0.1325"/>  <!-- 215 mm -->
   <!-- Slight outside offset so wheels stick out correctly -->
   <xacro:property name="wheel_y_offset" value="${W/2 + wheel_w/2 + 0.02}"/>
@@ -156,42 +182,44 @@
     <origin xyz="0.13 0.01 0.24" rpy="0 0 0"/>
   </joint>
-  <!-- Camera link + optical frame -->
-  <link name="camera_link">
-    <visual>
-      <!-- small housing placed on the front of the rover -->
+  <xacro:if value="false">
+    <!-- Camera link + optical frame -->
+    <link name="camera_link">
+      <visual>
+        <!-- small housing placed on the front of the rover -->
+        <origin xyz="0 0 0" rpy="0 0 0"/>
+        <geometry>
+          <box size="0.08 0.05 0.04"/>
+        </geometry>
+        <material name="black"><color rgba="0.0 0.0 0.0 1"/></material>
+      </visual>
+      <collision>
+        <origin xyz="0 0 0" rpy="0 0 0"/>
+        <geometry>
+          <box size="0.08 0.05 0.04"/>
+        </geometry>
+      </collision>
+      <inertial>
+        <mass value="0.2"/>
+        <origin xyz="0 0 0" rpy="0 0 0"/>
+        <inertia ixx="0.0005" ixy="0.0" ixz="0.0" iyy="0.0005" iyz="0.0" izz="0.0005"/>
+      </inertial>
+    </link>
+    <!-- Camera optical frame (use this frame for image topic) -->
+    <link name="camera_optical_frame"/>
+    <!-- Camera mount joint -->
+    <joint name="camera_joint" type="fixed">
+      <parent link="base_link"/>
+      <child link="camera_link"/>
+      <!-- placed on front-center at top; facing forward horizontally -->
+      <origin xyz="0.13 0 0.45" rpy="0 0 0"/>
+    </joint>
+    <!-- Optical frame fixed to camera_link (allows correct TF for image viewer/rviz) -->
+    <joint name="camera_to_optical" type="fixed">
+      <parent link="camera_link"/>
+      <child link="camera_optical_frame"/>
+      <!-- keep identity transform; change rpy if you need optical axes rotated -->
       <origin xyz="0 0 0" rpy="0 0 0"/>
-      <geometry>
-        <box size="0.08 0.05 0.04"/>
-      </geometry>
-      <material name="black"><color rgba="0.0 0.0 0.0 1"/></material>
-    </visual>
-    <collision>
-      <origin xyz="0 0 0" rpy="0 0 0"/>
-      <geometry>
-        <box size="0.08 0.05 0.04"/>
-      </geometry>
-    </collision>
-    <inertial>
-      <mass value="0.2"/>
-      <origin xyz="0 0 0" rpy="0 0 0"/>
-      <inertia ixx="0.0005" ixy="0.0" ixz="0.0" iyy="0.0005" iyz="0.0" izz="0.0005"/>
-    </inertial>
-  </link>
-  <!-- Camera optical frame (use this frame for image topic) -->
-  <link name="camera_optical_frame"/>
-  <!-- Camera mount joint -->
-  <joint name="camera_joint" type="fixed">
-    <parent link="base_link"/>
-    <child link="camera_link"/>
-    <!-- placed on front-center at top; facing forward horizontally -->
-    <origin xyz="0.13 0 0.45" rpy="0 0 0"/>
-  </joint>
-  <!-- Optical frame fixed to camera_link (allows correct TF for image viewer/rviz) -->
-  <joint name="camera_to_optical" type="fixed">
-    <parent link="camera_link"/>
-    <child link="camera_optical_frame"/>
-    <!-- keep identity transform; change rpy if you need optical axes rotated -->
-    <origin xyz="0 0 0" rpy="0 0 0"/>
-  </joint>
+    </joint>
+  </xacro:if>
   <!-- ========================= -->
   <!-- FOUR WHEELS -->
@@ -288,22 +316,24 @@
     </sensor>
   </gazebo>
-  <!-- Camera sensor attached to camera_link -->
-  <gazebo reference="camera_link">
-    <sensor name="camera_sensor" type="camera">
-      <topic>camera/image_raw</topic>
-      <update_rate>30</update_rate>
-      <camera>
-        <horizontal_fov>1.047</horizontal_fov>
-        <image>
-          <width>640</width>
-          <height>480</height>
-          <format>R8G8B8</format>
-        </image>
-        <clip>
-          <near>0.1</near>
-          <far>50.0</far>
-        </clip>
-      </camera>
-    </sensor>
-  </gazebo>
+  <xacro:if value="false">
+    <!-- Camera sensor attached to camera_link -->
+    <gazebo reference="camera_link">
+      <sensor name="camera_sensor" type="camera">
+        <topic>camera/image_raw</topic>
+        <update_rate>30</update_rate>
+        <camera>
+          <horizontal_fov>1.047</horizontal_fov>
+          <image>
+            <width>640</width>
+            <height>480</height>
+            <format>R8G8B8</format>
+          </image>
+          <clip>
+            <near>0.1</near>
+            <far>50.0</far>
+          </clip>
+        </camera>
+      </sensor>
+    </gazebo>
+  </xacro:if>
 </robot>

Commit message: Setting up some additional changes, i did with the launch and wifi reader files, SHOULD WORK NOW.

File: src/rover_description/urdf/robot.xacro (robot description, xacro)
@@ -1,28 +1,2 @@
-<!--I need to make sure a few things :
-the lidar_link visuals is flipped | pi value present, need to change that
-| The lidar z height is at 0.24, which is not good, need to change it :
-In your current code:
-- clearance is 0.1325 (Ground to bottom of chassis).
-- wheel_r is 0.05.
-- lidar_joint origin is at z="0.24".
-This means your LiDAR is positioned 0.24 meters above the base_link origin.
-The Problem: In your base_link visual/collision tags, you have the box offset by ${wheel_r + clearance + H/2}. In ROS, the base_link origin should ideally be on the floor or the center of the axles. Your current setup has the LiDAR floating quite high.
-The Fix: Use a relative property for the Lidar height so that when the chassis moves, the Lidar moves with it.
-and the imu:
-You have the IMU at xyz="0.13 0.01 0.24".
-As we discussed, if the IMU is offset from the center, the EKF has to do complex math to compensate for the "swing" when the robot rotates.
-The Fix: Move it to 0 0 0 (relative to the chassis) for now.
-updated code u can use:
-<joint name="imu_joint" type="fixed">
-    <parent link="base_link"/>
-    <child link="imu_link"/>
-    <origin xyz="0 0 0.05" rpy="0 0 0"/>
-  </joint>
-  <joint name="lidar_joint" type="fixed">
-    <parent link="base_link"/>
-    <child link="lidar_link"/>
-    <origin xyz="0.13 0 0.20" rpy="0 0 0"/>
-  </joint>
--->
 <?xml version="1.0"?>
 <robot xmlns:xacro="http://www.ros.org/wiki/xacro" name="four_wheel_rover">

Commit message: PHASE1 RECHECKING

File: src/rover_description/urdf/robot.xacro (robot description, xacro)
@@ -7,5 +7,5 @@
   <xacro:property name="W" value="0.290"/>     <!-- width -->
   <xacro:property name="H" value="0.160"/>     <!-- height -->
-  <xacro:property name="wheel_r" value="0.05"/>  <!-- radius -->
+  <xacro:property name="wheel_r" value="0.07"/>  <!-- radius 7cm (14cm diameter) -->
   <xacro:property name="wheel_w" value="0.08"/>  <!-- width -->
   <xacro:property name="clearance" value="0.1325"/>  <!-- 215 mm -->
@@ -100,5 +100,5 @@
         <origin xyz="0 0 0" rpy="${mesh_rpy}"/>
         <geometry>
-          <mesh filename="${mesh_stl}"/>
+          <mesh filename="${mesh_stl}" scale="1.4 1.4 1.4"/>
         </geometry>
       </visual>
@@ -132,5 +132,5 @@
   <link name="lidar_link">
     <visual>
-      <origin xyz="0 0 0" rpy="3.14159 0 0"/>
+      <origin xyz="0 0 0" rpy="0 0 0"/>
       <geometry>
           <mesh filename="package://rover_description/meshes/Lidar.STL" scale="1 1 1"/>
@@ -138,5 +138,5 @@
     </visual>
     <collision>
-      <origin xyz="0 0 0" rpy="3.14159 0 0"/>
+      <origin xyz="0 0 0" rpy="0 0 0"/>
       <geometry>
         <cylinder radius="0.065" length="0.05"/>
@@ -145,5 +145,5 @@
     <inertial>
       <mass value="0.3"/>
-      <origin xyz="0 0 0" rpy="3.14159 0 0"/>
+      <origin xyz="0 0 0" rpy="0 0 0"/>
       <inertia ixx="0.001" ixy="0.0" ixz="0.0" iyy="0.001" iyz="0.0" izz="0.001"/>
     </inertial>
@@ -154,5 +154,5 @@
     <child link="lidar_link"/>
     <!-- Mount at front-center of rover, facing forward horizontally -->
-    <origin xyz="0.13 0.01 0.24" rpy="0 0 0"/>
+    <origin xyz="0.23 -0.01 0.21" rpy="0 0 0"/>
   </joint>
   <xacro:if value="false">
@@ -186,5 +186,5 @@
       <child link="camera_link"/>
       <!-- placed on front-center at top; facing forward horizontally -->
-      <origin xyz="0.13 0 0.45" rpy="0 0 0"/>
+      <origin xyz="0.13 -0.01 0.45" rpy="0 0 0"/>
     </joint>
     <!-- Optical frame fixed to camera_link (allows correct TF for image viewer/rviz) -->
